File: PLL/PLL.kicad_sch (KiCad schematic)
At the start: 93 parts, among them M1 pch, M10 nch, M11 nch, M12 pch, M15 nch, M16 pch, M2 pch, M3 nch, M4 nch, M4 pch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

Commit message: Added missing files
Parts:
- added C?: 4p, symbol Device:C_Small
- Cp: value 9.35pF -> 9.33pF
- U1, U2: value 60uA -> 30uA
- renumbered Rs to R
Connections:
- net +1.2V: now also C?.2
- net VCONT: now also Cp.2, R.1
- net at U?. (out): now also U?. (out); no longer U?. (out)
- net at M?. (S), M?. (S): now also M?. (S), M?. (S); no longer M?. (S), M?. (S)
- net at U?. (~{Q}): no longer U?. (out)
- net at U?. (~{Q}): no longer U?. (~{Q})
- net at U?. (~{Q}): now also U?. (~{Q})
- new net: U?. (out), U?. (out)
- new net: C?.1, L?.1, M?. (S), M?. (S), M?. (S), M?. (S)
- new net: M?. (S), M?. (S), M?. (S), M?. (S), R?.1
- new net: M12. (S), M16. (S), U2. (plus)
- new net: M10. (S), M9. (S)
- new net: M4. (S), M5. (S)
- new net: M6. (S), M7. (S)
- new net: M1. (S), M2. (S)
- new net: M?. (S), M?. (S), M?. (S), M?. (S)
- new net: U?. (out), U?. (~{Q})
- new net: M15. (S), M3. (S), M4. (S)
- new net: M1. (S), M3. (S), U3. (out)
- new net: U?. (~{Q}), U?. (~{Q}) (x2)
- new net: M1. (S), M16. (S), M2. (S)
- new net: M11. (S), M15. (S), U1. (plus)
- now unconnected: U?. (~{Q}), U?. (~{Q})
